File: KiCad_projects/BPF/BPF.kicad_pcb (KiCad board)
At the start: 2 copper layers, 91 x 77.5 mm, 107 parts, among them J1 Barrel_Jack, J2 POWER, P10 CONN_01X01, P2 ANT/PA, P3 TRX, P5 CONN_01X06, P7 CONN_01X01, P8 CONN_01X01, P9 CONN_01X01, U1 74LS145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

Commit message: Fix Issues with PCB Silk Text
Other:
- board text added: "BPF US5NCJ ver. 1.05"
- board text removed: "PureSDR BPF ver. 1.04"
Changed lines of the file:
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@@
     (links 266)
     (no_connects 0)
-    (area 70.949999 43.449999 162.050001 121.050001)
+    (area 69.966667 40.866666 164.325001 121.825)
     (thickness 1.6)
     (drawings 14)
@@
   (page A4)
   (layers
-    (0 F.Cu signal)
-    (31 B.Cu signal)
+    (0 F.Cu signal hide)
+    (31 B.Cu signal hide)
     (32 B.Adhes user)
     (33 F.Adhes user)
@@
     (effects (font (size 1.5 1.5) (thickness 0.3)) (justify mirror))
   )
-  (gr_text "PureSDR BPF ver. 1.04\n" (at 138.2 118.16) (layer B.SilkS)
+  (gr_text "BPF US5NCJ  ver. 1.05\n" (at 138.2 118.16) (layer B.SilkS)
     (effects (font (size 1.5 1.5) (thickness 0.3)) (justify mirror))
   )
